File: Hardware/TempControl.sch (KiCad schematic (older format))
At the start: 32 parts, among them IC1 ATTINY84-SS, K1 S202S01, P1 Input, P2 Output, SW1 SPST, T1 BV030-7585.0, U1 MCP1802T, U2 DS18B20, X1 ISP, X2 20.0 MHz

Commit message: Standardized Schematics
Parts:
- removed R1, R2, R3, R4: 4.7kΩ, symbol SMALL_RESISTOR
- removed R5, R6: 300Ω, symbol SMALL_RESISTOR
- removed R7: 158Ω, symbol SMALL_RESISTOR
- removed R8: 47Ω, symbol SMALL_RESISTOR
- added R1, R2, R3, R4: 4.7k, symbol R
- added R5, R6: 300, symbol R
- added R7: 158, symbol R
- added R8: 47, symbol R
